File: kicad-project/pedale.kicad_pcb (KiCad board)
At the start: 2 copper layers, 121.5 x 81.5 mm, 45 parts, among them IC1 TLV76150DCYR, IC2 TLV76150DCYR, IC3 TLV76150DCYR, IC4 TLV76150DCYR, IC5 TLV76150DCYR

Commit message: modificari
Parts:
- R0, R1, R10, R11, R12, R13, R14, R2, R3, R4, R5, R6, R7, R8, R9: moved to F.Cu
- U1, U8: footprint Connector_PinHeader_2.54mm:PinHeader_1x02_P2.54mm_Vertical -> Connector_PinSocket_2.00mm:PinSocket_1x02_P2.00mm_Horizontal
- U2, U3, U5, U6, U7: footprint Connector_PinHeader_2.54mm:PinHeader_1x03_P2.54mm_Vertical -> Connector_PinSocket_2.00mm:PinSocket_1x03_P2.00mm_Horizontal
- moved C2 37.8 mm to (104.5, 45.0)
- moved C6 34.7 mm to (121.0, 78.0), turned to 0 degrees
- moved IC4 33.5 mm to (112.5, 78.0)
- moved C10 32.5 mm to (104.5, 79.5), turned to -90 degrees
- moved IC5 26.7 mm to (112.5, 43.5), turned to 180 degrees
- moved C7 20.4 mm to (104.5, 53.5), turned to -90 degrees
- moved IC1 19.4 mm to (112.5, 52.0)
- moved C3 18.8 mm to (121.0, 52.0), turned to 0 degrees
- moved C5 16.9 mm to (121.0, 69.0), turned to 0 degrees
- moved C1 16.6 mm to (121.0, 43.5)
- moved IC3 15.6 mm to (112.7, 69.0)
- moved R12 15.1 mm to (87.1, 48.0)
- moved U1 15.0 mm to (130.0, 62.0)
- moved R3 14.8 mm to (57.0, 48.0)
- moved R9 14.7 mm to (77.1, 48.0)
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Connections:
- net Net-(IC1-IN) renamed 12V
- net Net-(IC1-OUT_1) renamed /5V_2
- net Net-(IC2-OUT_1) renamed /5V_3
- net Net-(IC3-OUT_1) renamed /5V_4
- net Net-(IC4-OUT_1) renamed /5V_5
- net Net-(IC5-OUT_1) renamed /5V_1
- net Net-(U4-CANH) renamed /CAN_P
- net Net-(U4-CANL) renamed /CAN_N
- J13 pad 12: unconnected-(J13-GND-Pad12) -> GND
- J13 pad 14: unconnected-(J13-GND-Pad14) -> GND
Routing:
- net GND: track 218.9 -> 40.3 mm, vias 0 -> 20
- net /CAN_P: track 0.00 -> 112.8 mm
- net /CAN_N: track 0.00 -> 106.7 mm
- net /5V_5: track 0.00 -> 82.2 mm, vias 0 -> 1
- net /5V_4: track 0.00 -> 72.3 mm, vias 0 -> 1
- net /5V_3: track 0.00 -> 62.8 mm, vias 0 -> 1
- net /5V_2: track 0.00 -> 45.9 mm, vias 0 -> 1
- net /5V_1: track 0.00 -> 32.6 mm, vias 0 -> 1
- net 12V: track 78.7 -> 108.9 mm
- net Net-(J14-ptd1): track 51.7 -> 77.5 mm
- net Net-(U5-A0): track 40.1 -> 21.5 mm
- net Net-(J14-ptd0): track 44.7 -> 62.3 mm
- net Net-(J14-pta13): track 36.7 -> 53.3 mm
- net Net-(U3-A0): track 39.4 -> 24.9 mm
- net Net-(J14-pta9): track 29.8 -> 42.9 mm
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- added copper zone on F.Cu, net /5V_1
- added copper zone on F.Cu, net /5V_2
- added copper zone on F.Cu, net /5V_3
- added copper zone on F.Cu, net /5V_4
- added copper zone on F.Cu, net /5V_5
- added copper zone on F.Cu, net 12V
- added copper zone on B.Cu, net GND
- added copper zone on F.Cu, net GND
Other:
- outline, holes or cut-outs redrawn

Commit message: modificari 2
Routing:
- net GND: track 40.3 -> 34.8 mm
- net /5V_4: track 72.3 -> 72.9 mm
Changed lines of the file:
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@@
-	)
-	(segment
-		(start 106.22 34.66)
-		(end 106.22 31.78)
-		(width 1)
-		(layer "B.Cu")
-		(net 4)
-	)
-	(segment
-		(start 58.976 37.2)
-		(end 58.976 39.726)
-		(width 1)
-		(layer "B.Cu")
-		(net 4)
-	)
-	(segment
-		(start 58.976 39.726)
-		(end 59 39.75)
-		(width 1)
-		(layer "B.Cu")
-		(net 4)
 	)
 	(segment
@@
 	)
 	(segment
-		(start 60.175 31)
-		(end 68 31)
-		(width 0.25)
-		(layer "B.Cu")
-		(net 123)
-	)
-	(segment
-		(start 58.5 29.325)
-		(end 60.175 31)
-		(width 0.25)
-		(layer "B.Cu")
-		(net 123)
-	)
-	(segment
 		(start 69 40.25)
 		(end 97.75 69)
@@
 	)
 	(segment
+		(start 58.5 29.325)
+		(end 58.5 30.3)
+		(width 0.25)
+		(layer "B.Cu")
+		(net 123)
+	)
+	(segment
+		(start 58.5 30.3)
+		(end 59.2 31)
+		(width 0.25)
+		(layer "B.Cu")
+		(net 123)
+	)
+	(segment
 		(start 69 32)
 		(end 69 40.25)
@@
 		(start 97.75 69)
 		(end 107 69)
+		(width 0.25)
+		(layer "B.Cu")
+		(net 123)
+	)
+	(segment
+		(start 59.2 31)
+		(end 68 31)
 		(width 0.25)
 		(layer "B.Cu")
@@
 			)
 		)
-	)
-	(zone
-		(net 0)
-		(net_name "")
-		(layer "B.Cu")
-		(hatch edge 0.5)
-		(connect_pads
-			(clearance 0)
-		)
-		(min_thickness 0.25)
-		(filled_areas_thickness no)
-		(keepout
-			(tracks allowed)
-			(vias allowed)
-			(pads allowed)
-			(copperpour not_allowed)
-			(footprints allowed)
-		)
-		(placement
-			(enabled no)
-			(sheetname "/")
-		)
-		(fill
-			(thermal_gap 0.5)
-			(thermal_bridge_width 0.5)
-		)
-		(polygon
-			(pts
-				(xy 118.25 32.75) (xy 41.75 32.75) (xy 41.75 39.25) (xy 118.25 39.25)
-			)
-		)

Commit message: Schimbari dupa sugestii noi
Parts:
- removed U9: ~, Connector_PinHeader_2.54mm:PinHeader_1x01_P2.54mm_Vertical
- moved U8 104.2 mm to (26.3, 66.7), turned to 0 degrees
- moved U3 62.8 mm to (26.3, 38.5), turned to 0 degrees
- moved U7 58.8 mm to (26.8, 84.0), turned to 0 degrees
- moved U6 56.4 mm to (26.8, 76.0), turned to 0 degrees
- moved U2 55.1 mm to (26.3, 47.0), turned to 0 degrees
- moved U5 49.7 mm to (26.3, 55.2), turned to 0 degrees
Connections:
- J13 pad 12: GND -> unconnected-(J13-GND-Pad12)
- J13 pad 14: GND -> unconnected-(J13-GND-Pad14)
- J13 pad 16: unconnected-(J13-VBAT-Pad16) -> 12V
- J2 pad 7: GND -> unconnected-(J2-GND-Pad7)
- J4 pad 10: GND -> unconnected-(J4-GND-Pad10)
Routing:
- net /CAN_P: track 112.8 -> 5.64 mm
- net /CAN_N: track 106.7 -> 5.46 mm
- net Net-(U2-A0): track 40.6 -> 0.00 mm
- net Net-(U7-A0): track 27.3 -> 64.8 mm
- net Net-(U5-A0): track 21.5 -> 58.1 mm
- net Net-(U6-A0): track 38.5 -> 67.4 mm
- net 12V: track 108.9 -> 84.5 mm
- net Net-(U3-A0): track 24.9 -> 1.00 mm
- net Net-(J14-ptd1): track 77.5 -> 67.1 mm
- net Net-(J14-pta13): track 53.3 -> 54.8 mm
- net GND: vias 20 -> 16

Commit message: modificari aplicate
Parts:
- moved R0 22.0 mm to (46.5, 70.0)
- moved R3 22.0 mm to (57.0, 70.0)
- moved R6 22.0 mm to (66.5, 70.0)
- moved R12 15.0 mm to (87.0, 63.0)
- moved R9 15.0 mm to (77.0, 63.0)
- moved R11 8.00 mm to (77.0, 55.0), turned to 0 degrees
- moved R14 8.00 mm to (87.1, 55.0), turned to 0 degrees
- moved R10 7.00 mm to (77.0, 48.0), turned to 180 degrees
- moved R13 7.00 mm to (87.1, 48.0), turned to 180 degrees
- moved R2 1.00 mm to (46.5, 62.0), turned to 0 degrees
- moved R5 1.00 mm to (57.0, 62.0), turned to 0 degrees
- moved R8 1.00 mm to (66.5, 62.0), turned to 0 degrees
- turned R1 to 180 degrees
- turned R4 to 180 degrees
- turned R7 to 180 degrees
Connections:
- R0 pad 1: Net-(U7-A0) -> Net-(J14-ptd1)
- R0 pad 2: Net-(J14-ptd1) -> GND
- R1 pad 1: Net-(J14-ptd1) -> Net-(U7-A0)
- R10 pad 1: Net-(J14-pta8) -> Net-(U2-A0)
- R11 pad 2: GND -> Net-(J14-pta8)
- R12 pad 1: Net-(U3-A0) -> Net-(J14-pta9)
- R12 pad 2: Net-(J14-pta9) -> GND
- R13 pad 1: Net-(J14-pta9) -> Net-(U3-A0)
- R14 pad 2: GND -> Net-(J14-pta9)
- R2 pad 2: GND -> Net-(J14-ptd1)
- R3 pad 1: Net-(U6-A0) -> Net-(J14-ptd0)
- R3 pad 2: Net-(J14-ptd0) -> GND
- R4 pad 1: Net-(J14-ptd0) -> Net-(U6-A0)
- R5 pad 2: GND -> Net-(J14-ptd0)
- R6 pad 1: Net-(U5-A0) -> Net-(J14-pta13)
- R6 pad 2: Net-(J14-pta13) -> GND
- R7 pad 1: Net-(J14-pta13) -> Net-(U5-A0)
- R8 pad 2: GND -> Net-(J14-pta13)
- R9 pad 1: Net-(U2-A0) -> Net-(J14-pta8)
- R9 pad 2: Net-(J14-pta8) -> GND
Routing:
- net Net-(U3-A0): track 1.00 -> 68.6 mm
- net Net-(U2-A0): track 0.00 -> 59.7 mm
- net /5V_1: track 32.6 -> 85.4 mm
- net /5V_2: track 45.9 -> 85.1 mm
- net /5V_3: track 62.8 -> 85.2 mm
- net Net-(J14-ptd0): track 62.1 -> 43.6 mm
- net Net-(J14-pta13): track 54.8 -> 36.6 mm
- net Net-(J14-ptd1): track 67.1 -> 51.6 mm
- net /5V_4: track 72.9 -> 85.6 mm
- net Net-(J14-pta8): track 46.5 -> 35.8 mm
- net Net-(J14-pta9): track 42.9 -> 34.4 mm
- net Net-(U7-A0): track 64.8 -> 58.3 mm
- net Net-(U6-A0): track 67.4 -> 65.5 mm
- net Net-(R7-Pad2): track 8.00 -> 7.00 mm
- net Net-(R4-Pad2): track 8.00 -> 7.00 mm
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